File: Miniscope-v4-Dual-LED-ETL-Driver/KiCad/MS_v4_ETL_LED_Driver.sch (KiCad schematic (older format))
At the start: 32 parts, among them J1 Conn_01x01, J10 Conn_01x05, J6 Conn_01x01, J7 Conn_01x01, U1 MAX14574EWL+, U2 TPL0102-100RUCR, U3 LTC3218, U4 LTC3218

Commit message: Corrections
Fixed errors:

* Overlapping courtyards
* Traces very close to pads
* Bypass capacitors closer to pads
* Some courtyards (resistors/capacitors) had an error with the crosshairs. While not an important error it was fixed for easier debugging.
* Changed the symbol in the schematics for more consistency
To do

* Check the position of the LEDs relative to the miniscope
* Pour polygons planes in the LED ground pads
* Change the 3V3 and GND layer order
Parts:
- R5, R6, R7, R8: symbol Device:R_US -> .Resistor:ERJ-1GEF1022C
Changed lines of the file:
@@
 	1    0    0    -1
-$EndComp
-$Comp
-L .LED:LXZ1-PR01 D2
-U 1 1 5C198A03
-P 2550 1925
-F 0 "D2" V 2600 1875 50  0000 R CNN
-F 1 "LXZ1-PR01 (Blue)" V 2450 1925 50  0000 R CNN
-F 2 ".LED:LED_LXZ1_PR01_L" V 2550 1925 50  0001 C CNN
-F 3 "https://www.lumileds.com/uploads/415/DS105-pdf" V 2550 1925 50  0001 C CNN
-	1    2550 1925
-	0    -1   -1   0
 $EndComp
 Wire Wire Line
@@
 	6000 5375 8400 5375
 $Comp
-L Device:R_US R5
+L .Resistor:ERJ-1GEF1022C R5
 U 1 1 5D0314EF
 P 9100 1100
@@
 $EndComp
 $Comp
-L Device:R_US R6
-U 1 1 5D031D7C
-P 9100 1525
-F 0 "R6" H 9168 1571 50  0000 L CNN
-F 1 "4k7" H 9168 1480 50  0000 L CNN
-F 2 ".Resistor:R_0201_0603Metric_ERJ_L" V 9140 1515 50  0001 C CNN
-F 3 "~" H 9100 1525 50  0001 C CNN
-	1    9100 1525
-	1    0    0    -1
-$EndComp
-$Comp
-L Device:R_US R7
+L .Resistor:ERJ-1GEF1022C R7
 U 1 1 5D034890
 P 9950 1100
@@
 	1    0    0    -1
 $EndComp
-Wire Wire Line
-	9100 1675 9100 1775
-Wire Wire Line
-	9100 1250 9100 1325
-Wire Wire Line
-	9950 1250 9950 1300
 $Comp
 L power:+3.3V #PWR0111
@@
 	1    0    0    -1
 $EndComp
-Wire Wire Line
-	9100 850  9100 950
-Wire Wire Line
-	9950 850  9950 950
 Text Label 8750 1325 0    50   ~ 0
 Va
@@
 	8750 1325 9100 1325
 Connection ~ 9100 1325
-Wire Wire Line
-	9100 1325 9100 1375
 Text Label 9650 1300 0    50   ~ 0
 Vb
@@
 	9650 1300 9950 1300
 Connection ~ 9950 1300
-Wire Wire Line
-	9950 1300 9950 1375
 Wire Wire Line
 	5300 1575 5650 1575
@@
 _Wa
 $Comp
-L Device:R_US R8
+L .Resistor:ERJ-1GEF1022C R8
 U 1 1 5D07CC2E
 P 9950 1525
@@
 	1    0    0    -1
 $EndComp
-Wire Wire Line
-	9950 1675 9950 1775
 $Comp
 L Mechanical:MountingHole_Pad H1
@@
 Text Label 3925 2925 0    50   ~ 0
 _Wb
+$Comp
+L .LED:LXZ1-PR01 D2
+U 1 1 5D0BA34D
+P 2550 1925
+F 0 "D2" V 2596 1857 50  0000 R CNN
+F 1 "LXZ1-PR01 (Blue)" V 2505 1857 50  0000 R CNN
+F 2 ".LED:LED_LXZ1_PR01_L" H 2400 1950 50  0001 C CNN
+F 3 "https://www.lumileds.com/uploads/415/DS105-pdf" V 2550 1925 50  0001 C CNN
+	1    2550 1925
+	0    -1   -1   0
+$EndComp
+Wire Wire Line
+	9100 850  9100 1000
+Wire Wire Line
+	9100 1200 9100 1325
+$Comp
+L .Resistor:ERJ-1GEF1022C R6
+U 1 1 5D031D7C
+P 9100 1525
+F 0 "R6" H 9168 1571 50  0000 L CNN
+F 1 "4k7" H 9168 1480 50  0000 L CNN
+F 2 ".Resistor:R_0201_0603Metric_ERJ_L" V 9140 1515 50  0001 C CNN
+F 3 "~" H 9100 1525 50  0001 C CNN
+	1    9100 1525
+	1    0    0    -1
+$EndComp
+Wire Wire Line
+	9100 1325 9100 1425
+Wire Wire Line
+	9100 1625 9100 1775
+Wire Wire Line
+	9950 1200 9950 1300
+Wire Wire Line
+	9950 850  9950 1000
+Wire Wire Line
+	9950 1300 9950 1425
+Wire Wire Line
+	9950 1625 9950 1775
 $EndSCHEMATC

Commit message: Schematics update
Changes:

* Removed the pull-up 3k3 resistors in the I2C lines and replaced the with DNL value.
* Added the correct values for the voltage divider resistors

To do

* Fix the I2C resistors in the release board (wrongly placed as 10k2 resistors)
* Fix the position of LEDs and add two screws for better alignment
Parts:
- H1: footprint .Connector:Conn_1x1_100x100_Pad -> .Connector:Conn_1x1_700_Circular_Pad
- R1: Note 10.2K -> 10.2k
- R2, R3: value ERJ-1GEF1022C -> DNL
- R5, R7: value 8k2 -> ERJ-1GNJ622C; Note (none) -> 6.2k
- R6, R8: value 4k7 -> ERJ-1GEF3741C; Note (none) -> 3.74k
- U3, U4: symbol MS_v4_ETL_LED_Driver-rescue:LTC3218-.Driver_LED -> MS_v4_ETL_LED_Driver-rescue:LTC3218-.Driver_LED-MS_v4_ETL_LED_Driver-rescue
Changed lines of the file:
@@
 $EndComp
 $Comp
-L MS_v4_ETL_LED_Driver-rescue:LTC3218-.Driver_LED U3
+L MS_v4_ETL_LED_Driver-rescue:LTC3218-.Driver_LED-MS_v4_ETL_LED_Driver-rescue U3
 U 1 1 5C18A1DE
 P 1850 1675
@@
 F 2 ".Resistor:R_0201_0603Metric_ERJ_L" H 3230 2845 50  0001 C CNN
 F 3 "https://media.digikey.com/pdf/Data%20Sheets/Panasonic%20Resistors%20Thermistors%20PDFs/ERJ-G,R,E_Series_Rev_Oct_2014.pdf" H 3300 2925 50  0001 C CNN
-F 4 "10.2K" V 3186 2925 50  0000 C CNN "Note"
+F 4 "10.2k" V 3186 2925 50  0000 C CNN "Note"
 F 5 "0201" H 3530 3145 50  0001 C CNN "Size"
 	1    3300 2925
@@
 P 2850 7400
 F 0 "R3" V 2645 7400 50  0000 C CNN
-F 1 "ERJ-1GEF1022C" H 2880 7210 50  0001 L CNN
+F 1 "DNL" H 2880 7210 50  0001 L CNN
 F 2 ".Resistor:R_0201_0603Metric_ERJ_L" H 2780 7320 50  0001 C CNN
 F 3 "https://media.digikey.com/pdf/Data%20Sheets/Panasonic%20Resistors%20Thermistors%20PDFs/ERJ-G,R,E_Series_Rev_Oct_2014.pdf" H 2850 7400 50  0001 C CNN
@@
 P 2850 7150
 F 0 "R2" V 2645 7150 50  0000 C CNN
-F 1 "ERJ-1GEF1022C" H 2880 6960 50  0001 L CNN
+F 1 "DNL" H 2880 6960 50  0001 L CNN
 F 2 ".Resistor:R_0201_0603Metric_ERJ_L" H 2780 7070 50  0001 C CNN
 F 3 "https://media.digikey.com/pdf/Data%20Sheets/Panasonic%20Resistors%20Thermistors%20PDFs/ERJ-G,R,E_Series_Rev_Oct_2014.pdf" H 2850 7150 50  0001 C CNN
@@
 $EndComp
 $Comp
-L MS_v4_ETL_LED_Driver-rescue:LTC3218-.Driver_LED U4
+L MS_v4_ETL_LED_Driver-rescue:LTC3218-.Driver_LED-MS_v4_ETL_LED_Driver-rescue U4
 U 1 1 5D02BC5D
 P 4450 4125
@@
 	6000 5375 8400 5375
 $Comp
-L .Resistor:ERJ-1GEF1022C R5
-U 1 1 5D0314EF
-P 9100 1100
-F 0 "R5" H 9168 1146 50  0000 L CNN
-F 1 "8k2" H 9168 1055 50  0000 L CNN
-F 2 ".Resistor:R_0201_0603Metric_ERJ_L" V 9140 1090 50  0001 C CNN
-F 3 "~" H 9100 1100 50  0001 C CNN
-	1    9100 1100
-	1    0    0    -1
-$EndComp
-$Comp
 L .Resistor:ERJ-1GEF1022C R7
 U 1 1 5D034890
 P 9950 1100
 F 0 "R7" H 10018 1146 50  0000 L CNN
-F 1 "8k2" H 10018 1055 50  0000 L CNN
+F 1 "ERJ-1GNJ622C" H 10018 1055 50  0001 L CNN
 F 2 ".Resistor:R_0201_0603Metric_ERJ_L" V 9990 1090 50  0001 C CNN
 F 3 "~" H 9950 1100 50  0001 C CNN
+F 4 "6.2k" H 9800 1100 50  0000 C CNN "Note"
 	1    9950 1100
 	1    0    0    -1
@@
 P 9950 1525
 F 0 "R8" H 10018 1571 50  0000 L CNN
-F 1 "4k7" H 10018 1480 50  0000 L CNN
+F 1 "ERJ-1GEF3741C" H 10018 1480 50  0001 L CNN
 F 2 ".Resistor:R_0201_0603Metric_ERJ_L" V 9990 1515 50  0001 C CNN
 F 3 "~" H 9950 1525 50  0001 C CNN
+F 4 "3.74k" H 9800 1525 50  0000 C CNN "Note"
 	1    9950 1525
 	1    0    0    -1
@@
 F 0 "H1" V 6412 6603 50  0000 C CNN
 F 1 "MountingHole_Pad" V 6321 6603 50  0000 C CNN
-F 2 ".Connector:Conn_1x1_100x100_Pad" H 6175 6600 50  0001 C CNN
+F 2 ".Connector:Conn_1x1_700_Circular_Pad" H 6175 6600 50  0001 C CNN
 F 3 "~" H 6175 6600 50  0001 C CNN
 	1    6175 6600
@@
 P 9100 1525
 F 0 "R6" H 9168 1571 50  0000 L CNN
-F 1 "4k7" H 9168 1480 50  0000 L CNN
+F 1 "ERJ-1GEF3741C" H 9168 1480 50  0001 L CNN
 F 2 ".Resistor:R_0201_0603Metric_ERJ_L" V 9140 1515 50  0001 C CNN
-F 3 "~" H 9100 1525 50  0001 C CNN
+F 3 "https://b2b-api.panasonic.eu/file_stream/pids/fileversion/1242" H 9100 1525 50  0001 C CNN
+F 4 "3.74k" H 8825 1525 50  0000 L CNN "Note"
 	1    9100 1525
 	1    0    0    -1
@@
 Wire Wire Line
 	9950 1625 9950 1775
+$Comp
+L .Resistor:ERJ-1GEF1022C R5
+U 1 1 5D0314EF
+P 9100 1100
+F 0 "R5" H 9168 1146 50  0000 L CNN
+F 1 "ERJ-1GNJ622C" H 9168 1055 50  0001 L CNN
+F 2 ".Resistor:R_0201_0603Metric_ERJ_L" V 9140 1090 50  0001 C CNN
+F 3 "~" H 9100 1100 50  0001 C CNN
+F 4 "6.2k" H 8975 1100 50  0000 C CNN "Note"
+	1    9100 1100
+	1    0    0    -1
+$EndComp
 $EndSCHEMATC
