File: Miniscope-v4-Dual-LED-ETL-Driver/KiCad/MS_v4_ETL_LED_Driver_v2.sch (KiCad schematic (older format))
At the start: 32 parts, among them J1 Conn_01x01, J10 Conn_01x05, J6 Conn_01x01, J7 Conn_01x01, U1 MAX14574EWL+, U2 TPL0102-100RUCR, U3 LTC3218, U4 LTC3218

Commit message: Dual color Miniscope rev. 2
Changes:

* Completely redesigned  the PCB outline to match the new excitation module.
* The LEDs now fit perfectly one the center of the excitation module hole (see Fusion360 screenshot)
* In this iteration capacitors are much closer to their corresponding pins
* Corrected the width of the excitation module (previous version was 4 mm, now corrected to 3.5 mm)
* The EWL pads now are aligned to the center of the excitation module

To do:

* Final check of connections/ power planes
* Stress test the excitation module
Parts:
- D2: value LXZ1-PR01 (Blue) -> LXZ1-PR01
- U3, U4: symbol MS_v4_ETL_LED_Driver-rescue:LTC3218-.Driver_LED-MS_v4_ETL_LED_Driver-rescue -> MS_v4_ETL_LED_Driver-rescue:LTC3218-.Driver_LED-MS_v4_ETL_LED_Driver-rescue-MS_v4_ETL_LED_Driver-rescue
Changed lines of the file:
@@
 EESchema Schematic File Version 4
-LIBS:MS_v4_ETL_LED_Driver-cache
 EELAYER 29 0
 EELAYER END
@@
 $EndComp
 $Comp
-L MS_v4_ETL_LED_Driver-rescue:LTC3218-.Driver_LED-MS_v4_ETL_LED_Driver-rescue U3
+L MS_v4_ETL_LED_Driver-rescue:LTC3218-.Driver_LED-MS_v4_ETL_LED_Driver-rescue-MS_v4_ETL_LED_Driver-rescue U3
 U 1 1 5C18A1DE
 P 1850 1675
@@
 $EndComp
 $Comp
-L MS_v4_ETL_LED_Driver-rescue:LTC3218-.Driver_LED-MS_v4_ETL_LED_Driver-rescue U4
+L MS_v4_ETL_LED_Driver-rescue:LTC3218-.Driver_LED-MS_v4_ETL_LED_Driver-rescue-MS_v4_ETL_LED_Driver-rescue U4
 U 1 1 5D02BC5D
 P 4450 4125
@@
 Text Label 3925 2925 0    50   ~ 0
 _Wb
-$Comp
-L .LED:LXZ1-PR01 D2
-U 1 1 5D0BA34D
-P 2550 1925
-F 0 "D2" V 2596 1857 50  0000 R CNN
-F 1 "LXZ1-PR01 (Blue)" V 2505 1857 50  0000 R CNN
-F 2 ".LED:LED_LXZ1_PR01_L" H 2400 1950 50  0001 C CNN
-F 3 "https://www.lumileds.com/uploads/415/DS105-pdf" V 2550 1925 50  0001 C CNN
-	1    2550 1925
-	0    -1   -1   0
-$EndComp
 Wire Wire Line
 	9100 850  9100 1000
@@
 	1    0    0    -1
 $EndComp
+$Comp
+L .LED:LXZ1-PR01 D2
+U 1 1 5DBAF281
+P 2550 1925
+F 0 "D2" V 2596 1857 50  0000 R CNN
+F 1 "LXZ1-PR01" V 2505 1857 50  0000 R CNN
+F 2 ".LED:LED_LXZ1_PR01_L" H 2400 1950 50  0001 C CNN
+F 3 "https://www.lumileds.com/uploads/415/DS105-pdf" V 2550 1925 50  0001 C CNN
+	1    2550 1925
+	0    -1   -1   0
+$EndComp
 $EndSCHEMATC
